Commit message: modify description file and rviz file

File: sensor_description/urdf/vlp16.urdf.xacro (robot description, xacro)
@@ -19,10 +19,10 @@
       <visual>
         <geometry>
-          <mesh filename="package://velodyne_description/meshes/VLP16_base_1.dae" />
+          <mesh filename="package://sensor_description/meshes/VLP16_base_1.dae" />
         </geometry>
       </visual>
       <visual>
         <geometry>
-          <mesh filename="package://velodyne_description/meshes/VLP16_base_2.dae" />
+          <mesh filename="package://sensor_description/meshes/VLP16_base_2.dae" />
         </geometry>
       </visual>
@@ -48,5 +48,5 @@
         <origin xyz="0 0 -0.0377" />
         <geometry>
-          <mesh filename="package://velodyne_description/meshes/VLP16_scan.dae" />
+          <mesh filename="package://sensor_description/meshes/VLP16_scan.dae" />
         </geometry>
       </visual>
