Commit message: modify urdf for stereo_camera and tf of image0

File: sensor_description/urdf/sensor_general.urdf.xacro (robot description, xacro)
@@ -5,9 +5,12 @@
   <xacro:property name="camera_diameter" value="0.1055" />
   <xacro:property name="camera_mass" value="1.128" />
-  <material name="gray">
-    <color rgba="0.4 0.4 0.4 1"/>
-  </material>
-  <material name="dark_gray">
-    <color rgba="0.2 0.2 0.2 1"/>
+  <!-- <material name="gray"> -->
+  <!--   <color rgba="0.4 0.4 0.4 1"/> -->
+  <!-- </material> -->
+  <!-- <material name="dark_gray"> -->
+  <!--   <color rgba="0.2 0.2 0.2 1"/> -->
+  <!-- </material> -->
+  <material name="blue">
+    <color rgba="0 0.4 0.8 1" />
   </material>
   <!-- Base Footprint -->
@@ -24,5 +27,5 @@
 	<cylinder length="${camera_height}" radius="${camera_diameter / 2}"/>
       </geometry>
-       <!-- <material name="gray"/> -->
+      <material name="blue"/>
     </visual>
     <!-- <collision> -->
@@ -54,4 +57,10 @@
     <!-- </inertial> -->
   </link>
+  <link name="image0" />
+  <joint name="camera_inside_joint" type="fixed">
+    <parent link="camera_foot" />
+    <child link ="image0" />
+    <origin xyz="${camera_diameter / 2} 0 ${(camera_height / 2) + 0.06}" rpy="0 0 0" />
+  </joint>
   <VLP-16 parent="camera_link" name="velodyne">
     <origin xyz="0 0 ${camera_height / 2}" rpy="0 0 0" />

Commit message: modify urdf for camera

File: sensor_description/urdf/sensor_general.urdf.xacro (robot description, xacro)
@@ -8,12 +8,12 @@
   </material>
   <!-- Base Footprint -->
-  <link name="base_footprint" />
+  <link name="camera_foot" />
   <!-- Base Link -->
   <joint name="footprint" type="fixed" >
-    <parent link="base_footprint" />
-    <child link="base_link" />
+    <parent link="camera_foot" />
+    <child link="camera_link" />
     <origin xyz="0 0 0.2" rpy="0 0 0" />
   </joint>
-  <link name="base_link" >
+  <link name="camera_link" >
     <visual>
       <geometry>
@@ -36,21 +36,6 @@
   </link>
   <xacro:include filename="$(find sensor_description)/urdf/vlp16.urdf.xacro"/>
-  <VLP-16 parent="base_link" name="velodyne">
+  <VLP-16 parent="camera_link" name="velodyne">
     <origin xyz="0 0 0.2" rpy="0 0 0" />
   </VLP-16>
-  <joint name="camera_joint" type="fixed" >
-    <!-- <origin xyz="0.048 0 0.315" rpy="0 0 0" /> -->
-    <!-- <origin xyz="0.048 0 0.315" rpy="-1.57 0 -1.57" /> -->
-    <origin xyz="0.048 0.17 0.315" rpy="-1.57 0 -1.57" />
-    <parent link="base_link" />
-    <child link="camera_link" />
-  </joint>
-  <link name="camera_link">
-    <visual>
-      <geometry>
-        <box size="0.09 0.03 0.02" />
-      </geometry>
-       <material name="dark_gray"/>
-    </visual>
-  </link>
 </robot>

File: sensor_description/urdf/vlp16.urdf.xacro (robot description, xacro)
@@ -2,12 +2,12 @@
 <robot xmlns:xacro="http://www.ros.org/wiki/xacro" name="VLP-16">
   <xacro:property name="M_PI" value="3.1415926535897931" />
-  <!-- <xacro:macro name="VLP-16" params="*origin parent:=base_link name:=velodyne topic:=/velodyne_points hz:=10 lasers:=16 samples:=1875 collision_range:=0.3 min_range:=0.9 max_range:=130.0 noise:=0.008 min_angle:=-${M_PI} max_angle:=${M_PI}"> -->
-  <xacro:macro name="VLP-16" params="*origin parent:=base_link name:=velodyne">
+  <!-- <xacro:macro name="VLP-16" params="*origin parent:=camera_link name:=velodyne topic:=/velodyne_points hz:=10 lasers:=16 samples:=1875 collision_range:=0.3 min_range:=0.9 max_range:=130.0 noise:=0.008 min_angle:=-${M_PI} max_angle:=${M_PI}"> -->
+  <xacro:macro name="VLP-16" params="*origin parent:=camera_link name:=velodyne">
     <joint name="${name}_base_mount_joint" type="fixed">
       <xacro:insert_block name="origin" />
       <parent link="${parent}"/>
-      <child link="${name}_base_link"/>
+      <child link="${name}_camera_link"/>
     </joint>
-    <link name="${name}_base_link">
+    <link name="${name}_camera_link">
       <inertial>
         <mass value="0.83"/>
@@ -36,5 +36,5 @@
     <joint name="${name}_base_scan_joint" type="fixed" >
       <origin xyz="0 0 0.0377" rpy="0 0 0" />
-      <parent link="${name}_base_link" />
+      <parent link="${name}_camera_link" />
       <child link="${name}"/>
     </joint>

Commit message: modify urdf for stereo_camera

File: sensor_description/urdf/sensor_general.urdf.xacro (robot description, xacro)
@@ -1,4 +1,8 @@
 <?xml version="1.0"?>
 <robot xmlns:xacro="http://www.ros.org/wiki/xacro" name="example">
+  <xacro:include filename="$(find sensor_description)/urdf/vlp16.urdf.xacro"/>
+  <xacro:property name="camera_height" value="0.1767" />
+  <xacro:property name="camera_diameter" value="0.1055" />
+  <xacro:property name="camera_mass" value="1.128" />
   <material name="gray">
     <color rgba="0.4 0.4 0.4 1"/>
@@ -13,29 +17,43 @@
     <parent link="camera_foot" />
     <child link="camera_link" />
-    <origin xyz="0 0 0.2" rpy="0 0 0" />
+    <origin xyz="0 0 ${camera_height / 2}" rpy="0 0 0" />
   </joint>
   <link name="camera_link" >
     <visual>
       <geometry>
-        <box size="0.15 0.15 0.4" />
+	<cylinder length="${camera_height}" radius="${camera_diameter / 2}"/>
       </geometry>
-       <material name="gray"/>
+       <!-- <material name="gray"/> -->
     </visual>
-    <collision>
-      <geometry>
-        <box size="0.15 0.15 0.4" />
-      </geometry>
-    </collision>
-    <inertial>
-      <origin xyz="0 0 0"/>
-      <mass value="10"/>
-      <inertia ixx="3.0" ixy="0.0" ixz="0.0"
-               iyy="3.0" iyz="0.0"
-               izz="3.0" />
-    </inertial>
+    <!-- <collision> -->
+    <!--   <geometry> -->
+    <!--     <box size="0.15 0.15 0.4" /> -->
+    <!--   </geometry> -->
+    <!-- </collision> -->
+    <!-- <inertial> -->
+    <!--   <origin xyz="0 0 0"/> -->
+    <!--   <mass value="10"/> -->
+    <!--   <inertia ixx="3.0" ixy="0.0" ixz="0.0" -->
+    <!--            iyy="3.0" iyz="0.0" -->
+    <!--            izz="3.0" /> -->
+    <!-- </inertial> -->
+    <!-- <visual> -->
+    <!--   <geometry> -->
+    <!--     <cylinder length="${camera_height}" radius="${camera_radius}" /> -->
+    <!--   </geometry> -->
+    <!--   <material name="gray"/> -->
+    <!-- </visual> -->
+    <!-- <collision> -->
+    <!--   <geometry> -->
+    <!--     <cylinder length="${camera_height}" radius="${camera_radius}"/> -->
+    <!--   </geometry> -->
+    <!-- </collision> -->
+    <!-- <inertial> -->
+    <!--   <origin xyz="0 0 0"/> -->
+    <!--   <mass value="${camera_mass}"/> -->
+    <!-- </inertial> -->
   </link>
-  <xacro:include filename="$(find sensor_description)/urdf/vlp16.urdf.xacro"/>
   <VLP-16 parent="camera_link" name="velodyne">
-    <origin xyz="0 0 0.2" rpy="0 0 0" />
+    <origin xyz="0 0 ${camera_height / 2}" rpy="0 0 0" />
   </VLP-16>
 </robot>

File: sensor_description/urdf/vlp16.urdf.xacro (robot description, xacro)
@@ -1,6 +1,4 @@
 <?xml version="1.0"?>
 <robot xmlns:xacro="http://www.ros.org/wiki/xacro" name="VLP-16">
-  <xacro:property name="M_PI" value="3.1415926535897931" />
-  <!-- <xacro:macro name="VLP-16" params="*origin parent:=camera_link name:=velodyne topic:=/velodyne_points hz:=10 lasers:=16 samples:=1875 collision_range:=0.3 min_range:=0.9 max_range:=130.0 noise:=0.008 min_angle:=-${M_PI} max_angle:=${M_PI}"> -->
   <xacro:macro name="VLP-16" params="*origin parent:=camera_link name:=velodyne">
     <joint name="${name}_base_mount_joint" type="fixed">

Commit message: modigy urdf for stereo_camera omni

File: sensor_description/urdf/sensor_general.urdf.xacro (robot description, xacro)
@@ -2,66 +2,6 @@
 <robot xmlns:xacro="http://www.ros.org/wiki/xacro" name="example">
   <xacro:include filename="$(find sensor_description)/urdf/vlp16.urdf.xacro"/>
-  <xacro:property name="camera_height" value="0.1767" />
-  <xacro:property name="camera_diameter" value="0.1055" />
-  <xacro:property name="camera_mass" value="1.128" />
-  <!-- <material name="gray"> -->
-  <!--   <color rgba="0.4 0.4 0.4 1"/> -->
-  <!-- </material> -->
-  <!-- <material name="dark_gray"> -->
-  <!--   <color rgba="0.2 0.2 0.2 1"/> -->
-  <!-- </material> -->
-  <material name="blue">
-    <color rgba="0 0.4 0.8 1" />
-  </material>
-  <!-- Base Footprint -->
-  <link name="camera_foot" />
-  <!-- Base Link -->
-  <joint name="footprint" type="fixed" >
-    <parent link="camera_foot" />
-    <child link="camera_link" />
-    <origin xyz="0 0 ${camera_height / 2}" rpy="0 0 0" />
-  </joint>
-  <link name="camera_link" >
-    <visual>
-      <geometry>
-	<cylinder length="${camera_height}" radius="${camera_diameter / 2}"/>
-      </geometry>
-      <material name="blue"/>
-    </visual>
-    <!-- <collision> -->
-    <!--   <geometry> -->
-    <!--     <box size="0.15 0.15 0.4" /> -->
-    <!--   </geometry> -->
-    <!-- </collision> -->
-    <!-- <inertial> -->
-    <!--   <origin xyz="0 0 0"/> -->
-    <!--   <mass value="10"/> -->
-    <!--   <inertia ixx="3.0" ixy="0.0" ixz="0.0" -->
-    <!--            iyy="3.0" iyz="0.0" -->
-    <!--            izz="3.0" /> -->
-    <!-- </inertial> -->
-    <!-- <visual> -->
-    <!--   <geometry> -->
-    <!--     <cylinder length="${camera_height}" radius="${camera_radius}" /> -->
-    <!--   </geometry> -->
-    <!--   <material name="gray"/> -->
-    <!-- </visual> -->
-    <!-- <collision> -->
-    <!--   <geometry> -->
-    <!--     <cylinder length="${camera_height}" radius="${camera_radius}"/> -->
-    <!--   </geometry> -->
-    <!-- </collision> -->
-    <!-- <inertial> -->
-    <!--   <origin xyz="0 0 0"/> -->
-    <!--   <mass value="${camera_mass}"/> -->
-    <!-- </inertial> -->
-  </link>
-  <link name="image0" />
-  <joint name="camera_inside_joint" type="fixed">
-    <parent link="camera_foot" />
-    <child link ="image0" />
-    <origin xyz="${camera_diameter / 2} 0 ${(camera_height / 2) + 0.06}" rpy="0 0 0" />
-  </joint>
-  <VLP-16 parent="camera_link" name="velodyne">
+  <xacro:include filename="$(find sensor_description)/urdf/occam.urdf.xacro"/>
+  <VLP-16 parent="occam" name="velodyne">
     <origin xyz="0 0 ${camera_height / 2}" rpy="0 0 0" />
   </VLP-16>
